File: testBoard/testBoard/testBoard.kicad_pcb (KiCad board)
At the start: 2 copper layers, 3 parts

Commit message: Intermediate
Parts:
- added REF**: SOT-23, Package_TO_SOT_SMD:SOT-23, F.Cu at (119.8, 107.5)
- added REF**: SOIC-14_3.9x8.7mm_P1.27mm, Package_SO:SOIC-14_3.9x8.7mm_P1.27mm, F.Cu at (110.8, 103.9)
Routing:
- net (no net): track 49.4 -> 126.4 mm
Changed lines of the file:
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@@
     (thickness 1.6)
     (drawings 0)
-    (tracks 5)
+    (tracks 35)
     (zones 0)
-    (modules 3)
+    (modules 5)
     (nets 1)
   )
@@
   )
   (setup
-    (last_trace_width 1)
+    (last_trace_width 0.5)
+    (user_trace_width 0.5)
     (user_trace_width 1)
     (trace_clearance 0.2)
@@
     (mod_text_size 1 1)
     (mod_text_width 0.15)
-    (pad_size 1.524 1.524)
-    (pad_drill 0.762)
+    (pad_size 1.95 0.6)
+    (pad_drill 0)
     (pad_to_mask_clearance 0.051)
     (solder_mask_min_width 0.25)
     (aux_axis_origin 0 0)
-    (visible_elements FFFFFF7F)
+    (visible_elements 7FFFFFFF)
     (pcbplotparams
-      (layerselection 0x010fc_ffffffff)
+      (layerselection 0x00000_7fffffff)
       (usegerberextensions false)
       (usegerberattributes false)
       (usegerberadvancedattributes false)
-      (creategerberjobfile false)
+      (creategerberjobfile true)
       (excludeedgelayer true)
       (linewidth 0.100000)
@@
       (outputformat 1)
       (mirror false)
-      (drillshape 1)
+      (drillshape 0)
       (scaleselection 1)
       (outputdirectory ""))
@@
     (uvia_drill 0.1)
   )
+  (module Package_TO_SOT_SMD:SOT-23 (layer F.Cu)
+    (at 119.8 107.5)
+    (descr "SOT-23, Standard")
+    (tags SOT-23)
+    (attr smd)
+    (fp_text reference REF** (at 0 -2.5) (layer F.SilkS)
+      (effects (font (size 1 1) (thickness 0.15)))
+    )
+    (fp_text value SOT-23 (at 0 2.5) (layer F.Fab)
+      (effects (font (size 1 1) (thickness 0.15)))
+    )
+    (fp_line (start 0.76 1.58) (end -0.7 1.58) (layer F.SilkS) (width 0.12))
+    (fp_line (start 0.76 -1.58) (end -1.4 -1.58) (layer F.SilkS) (width 0.12))
+    (fp_line (start -1.7 1.75) (end -1.7 -1.75) (layer F.CrtYd) (width 0.05))
+    (fp_line (start 1.7 1.75) (end -1.7 1.75) (layer F.CrtYd) (width 0.05))
+    (fp_line (start 1.7 -1.75) (end 1.7 1.75) (layer F.CrtYd) (width 0.05))
+    (fp_line (start -1.7 -1.75) (end 1.7 -1.75) (layer F.CrtYd) (width 0.05))
+    (fp_line (start 0.76 -1.58) (end 0.76 -0.65) (layer F.SilkS) (width 0.12))
+    (fp_line (start 0.76 1.58) (end 0.76 0.65) (layer F.SilkS) (width 0.12))
+    (fp_line (start -0.7 1.52) (end 0.7 1.52) (layer F.Fab) (width 0.1))
+    (fp_line (start 0.7 -1.52) (end 0.7 1.52) (layer F.Fab) (width 0.1))
+    (fp_line (start -0.7 -0.95) (end -0.15 -1.52) (layer F.Fab) (width 0.1))
+    (fp_line (start -0.15 -1.52) (end 0.7 -1.52) (layer F.Fab) (width 0.1))
+    (fp_line (start -0.7 -0.95) (end -0.7 1.5) (layer F.Fab) (width 0.1))
+    (fp_text user %R (at 0 0 90) (layer F.Fab)
+      (effects (font (size 0.5 0.5) (thickness 0.075)))
+    )
+    (pad 3 smd rect (at 1 0) (size 0.9 0.8) (layers F.Cu F.Paste F.Mask))
+    (pad 2 smd rect (at -1 0.95) (size 0.9 0.8) (layers F.Cu F.Paste F.Mask))
+    (pad 1 smd rect (at -1 -0.95) (size 0.9 0.8) (layers F.Cu F.Paste F.Mask))
+    (model ${KISYS3DMOD}/Package_TO_SOT_SMD.3dshapes/SOT-23.wrl
+      (at (xyz 0 0 0))
+      (scale (xyz 1 1 1))
+      (rotate (xyz 0 0 0))
+    )
+  )
+  (module Package_SO:SOIC-14_3.9x8.7mm_P1.27mm (layer F.Cu)
+    (at 110.8 103.9)
+    (descr "SOIC, 14 Pin (JEDEC MS-012AB, https://www.analog.com/media/en/package-pcb-resources/package/pkg_pdf/soic_narrow-r/r_14.pdf), generated with kicad-footprint-generator ipc_gullwing_generator.py")
+    (tags "SOIC SO")
+    (attr smd)
+    (fp_text reference REF** (at 0 -5.28) (layer F.SilkS)
+      (effects (font (size 1 1) (thickness 0.15)))
+    )
+    (fp_text value SOIC-14_3.9x8.7mm_P1.27mm (at 0 5.28) (layer F.Fab)
+      (effects (font (size 1 1) (thickness 0.15)))
+    )
+    (fp_text user %R (at 0 0) (layer F.Fab)
+      (effects (font (size 0.98 0.98) (thickness 0.15)))
+    )
+    (fp_line (start 3.7 -4.58) (end -3.7 -4.58) (layer F.CrtYd) (width 0.05))
+    (fp_line (start 3.7 4.58) (end 3.7 -4.58) (layer F.CrtYd) (width 0.05))
+    (fp_line (start -3.7 4.58) (end 3.7 4.58) (layer F.CrtYd) (width 0.05))
+    (fp_line (start -3.7 -4.58) (end -3.7 4.58) (layer F.CrtYd) (width 0.05))
+    (fp_line (start -1.95 -3.35) (end -0.975 -4.325) (layer F.Fab) (width 0.1))
+    (fp_line (start -1.95 4.325) (end -1.95 -3.35) (layer F.Fab) (width 0.1))
+    (fp_line (start 1.95 4.325) (end -1.95 4.325) (layer F.Fab) (width 0.1))
+    (fp_line (start 1.95 -4.325) (end 1.95 4.325) (layer F.Fab) (width 0.1))
+    (fp_line (start -0.975 -4.325) (end 1.95 -4.325) (layer F.Fab) (width 0.1))
+    (fp_line (start 0 -4.435) (end -3.45 -4.435) (layer F.SilkS) (width 0.12))
+    (fp_line (start 0 -4.435) (end 1.95 -4.435) (layer F.SilkS) (width 0.12))
+    (fp_line (start 0 4.435) (end -1.95 4.435) (layer F.SilkS) (width 0.12))
+    (fp_line (start 0 4.435) (end 1.95 4.435) (layer F.SilkS) (width 0.12))
+    (pad 14 smd roundrect (at 2.475 -3.81) (size 1.95 0.6) (layers F.Cu F.Paste F.Mask) (roundrect_rratio 0.25))
+    (pad 13 smd roundrect (at 2.475 -2.54) (size 1.95 0.6) (layers F.Cu F.Paste F.Mask) (roundrect_rratio 0.25))
+    (pad 12 smd roundrect (at 2.475 -1.27) (size 1.95 0.6) (layers F.Cu F.Paste F.Mask) (roundrect_rratio 0.25))
+    (pad 11 smd roundrect (at 2.475 0) (size 1.95 0.6) (layers F.Cu F.Paste F.Mask) (roundrect_rratio 0.25))
+    (pad 10 smd roundrect (at 2.475 1.27) (size 1.95 0.6) (layers F.Cu F.Paste F.Mask) (roundrect_rratio 0.25))
+    (pad 9 smd rect (at 2.475 2.54) (size 1.95 0.6) (layers F.Cu F.Paste F.Mask))
+    (pad 8 smd roundrect (at 2.475 3.81) (size 1.95 0.6) (layers F.Cu F.Paste F.Mask) (roundrect_rratio 0.25))
+    (pad 7 smd roundrect (at -2.475 3.81) (size 1.95 0.6) (layers F.Cu F.Paste F.Mask) (roundrect_rratio 0.25))
+    (pad 6 smd roundrect (at -2.475 2.54) (size 1.95 0.6) (layers F.Cu F.Paste F.Mask) (roundrect_rratio 0.25))
+    (pad 5 smd roundrect (at -2.475 1.27) (size 1.95 0.6) (layers F.Cu F.Paste F.Mask) (roundrect_rratio 0.25))
+    (pad 4 smd roundrect (at -2.475 0) (size 1.95 0.6) (layers F.Cu F.Paste F.Mask) (roundrect_rratio 0.25))
+    (pad 3 smd roundrect (at -2.475 -1.27) (size 1.95 0.6) (layers F.Cu F.Paste F.Mask) (roundrect_rratio 0.25))
+    (pad 2 smd roundrect (at -2.475 -2.54) (size 1.95 0.6) (layers F.Cu F.Paste F.Mask) (roundrect_rratio 0.25))
+    (pad 1 smd roundrect (at -2.475 -3.81) (size 1.95 0.6) (layers F.Cu F.Paste F.Mask) (roundrect_rratio 0.25))
+    (model ${KISYS3DMOD}/Package_SO.3dshapes/SOIC-14_3.9x8.7mm_P1.27mm.wrl
+      (at (xyz 0 0 0))
+      (scale (xyz 1 1 1))
+      (rotate (xyz 0 0 0))
+    )
+  )
   (module Connector_Pin:Pin_D1.0mm_L10.0mm_LooseFit (layer F.Cu)
     (at 92.71 106.68)
@@
   (segment (start 113.03 87.63) (end 114.3 88.9) (width 1) (layer F.Cu) (net 0))
   (segment (start 92.71 95.25) (end 100.33 87.63) (width 1) (layer F.Cu) (net 0))
-  (segment (start 92.71 106.68) (end 92.71 95.25) (width 1) (layer F.Cu) (net 0))
   (segment (start 87.63 87.63) (end 100.33 87.63) (width 1) (layer F.Cu) (net 0))
   (segment (start 100.33 87.63) (end 113.03 87.63) (width 1) (layer F.Cu) (net 0))
+  (segment (start 94.31 100.09) (end 92.71 98.49) (width 0.5) (layer F.Cu) (net 0))
+  (segment (start 108.325 100.09) (end 94.31 100.09) (width 0.5) (layer F.Cu) (net 0))
+  (segment (start 92.71 106.68) (end 92.71 98.49) (width 1) (layer F.Cu) (net 0))
+  (segment (start 92.71 98.49) (end 92.71 95.25) (width 1) (layer F.Cu) (net 0))
+  (segment (start 113.275 102.63) (end 117.17 102.63) (width 0.5) (layer F.Cu) (net 0))
+  (segment (start 117.17 102.63) (end 117.7 102.1) (width 0.5) (layer F.Cu) (net 0))
+  (segment (start 117.7 102.1) (end 117.7 98.1) (width 0.5) (layer F.Cu) (net 0))
+  (segment (start 117.7 98.1) (end 114.1 94.5) (width 0.5) (layer F.Cu) (net 0))
+  (segment (start 114.3 94.3) (end 114.3 88.9) (width 0.5) (layer F.Cu) (net 0))
+  (segment (start 114.1 94.5) (end 114.3 94.3) (width 0.5) (layer F.Cu) (net 0))
+  (segment (start 108.325 106.44) (end 105.44 106.44) (width 0.5) (layer F.Cu) (net 0))
+  (segment (start 105.44 106.44) (end 104.5 105.5) (width 0.5) (layer F.Cu) (net 0))
+  (segment (start 104.5 105.5) (end 104.5 103.6) (width 0.5) (layer F.Cu) (net 0))
+  (segment (start 105.47 102.63) (end 108.325 102.63) (width 0.5) (layer F.Cu) (net 0))
+  (segment (start 104.5 103.6) (end 105.47 102.63) (width 0.5) (layer F.Cu) (net 0))
+  (segment (start 112.90429 99.71929) (end 111.38071 99.71929) (width 0.5) (layer F.Cu) (net 0))
+  (segment (start 113.275 100.09) (end 112.90429 99.71929) (width 0.5) (layer F.Cu) (net 0))
+  (segment (start 111.38071 99.71929) (end 110.9 100.2) (width 0.5) (layer F.Cu) (net 0))
+  (segment (start 110.9 100.2) (end 110.9 104.8) (width 0.5) (layer F.Cu) (net 0))
+  (segment (start 111.27 105.17) (end 113.275 105.17) (width 0.5) (layer F.Cu) (net 0))
+  (segment (start 110.9 104.8) (end 111.27 105.17) (width 0.5) (layer F.Cu) (net 0))
+  (segment (start 118.8 105.65) (end 118.8 106.55) (width 0.5) (layer F.Cu) (net 0))
+  (segment (start 117.05 103.9) (end 118.8 105.65) (width 0.5) (layer F.Cu) (net 0))
+  (segment (start 113.275 103.9) (end 117.05 103.9) (width 0.5) (layer F.Cu) (net 0))
+  (segment (start 108.69571 105.54071) (end 109.94071 105.54071) (width 0.5) (layer F.Cu) (net 0))
+  (segment (start 108.325 105.17) (end 108.69571 105.54071) (width 0.5) (layer F.Cu) (net 0))
+  (segment (start 109.94071 105.54071) (end 110.8 106.4) (width 0.5) (layer F.Cu) (net 0))
+  (segment (start 110.8 106.4) (end 110.8 108.7) (width 0.5) (layer F.Cu) (net 0))
+  (segment (start 110.8 108.7) (end 111.5 109.4) (width 0.5) (layer F.Cu) (net 0))
+  (segment (start 112.45 108.45) (end 118.8 108.45) (width 0.5) (layer F.Cu) (net 0))
+  (segment (start 111.5 109.4) (end 112.45 108.45) (width 0.5) (layer F.Cu) (net 0))
 )
